File: hw_rfid/hw_rfid.kicad_sch (KiCad schematic)
At the start: 46 parts, among them IC1 XC9288A33CER-G, IC2 TPS610333DRLR, J1 Conn_01x02, J2 Conn_01x05, J3 Conn_01x04, J4 Conn_01x03, J5 Conn_01x08, Q1 2N7002, SW1 SW_Push, SW2 SW_Push, SW3 SW_Push, U1 STM32U031K6Ux, U2 AT45DB021E-SHN-T

Commit message: feat: Changing the way of import the libs
Parts:
- IC1: footprint XC9288A:USP-6C -> AT45DB021E-SHN-T:SOIC127P798X216-8N
- IC2: footprint TPS6103:SOTFL50P160X60-8N -> TPS610333DRLR:SOTFL50P160X60-8N
- U2: footprint AT45DB:SOIC127P798X216-8N -> AT45DB021E-SHN-T:SOIC127P798X216-8N
Changed lines of the file:
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@@
 			)
 		)
-		(property "Footprint" "AT45DB:SOIC127P798X216-8N"
+		(property "Footprint" "AT45DB021E-SHN-T:SOIC127P798X216-8N"
 			(at 234.95 124.46 0)
 			(effects
@@
 			)
 		)
-		(property "Footprint" "TPS6103:SOTFL50P160X60-8N"
+		(property "Footprint" "TPS610333DRLR:SOTFL50P160X60-8N"
 			(at 218.44 143.18 0)
 			(effects
@@
 			)
 		)
-		(property "Footprint" "XC9288A:USP-6C"
+		(property "Footprint" "AT45DB021E-SHN-T:SOIC127P798X216-8N"
 			(at 137.16 127.94 0)
 			(effects

Commit message: PLACA atualizada
Parts:
- IC1: footprint AT45DB021E-SHN-T:SOIC127P798X216-8N -> XC9288A33CER-G:USP-6C
Connections:
- net LPUART2_RX: now also J3.2 (Pin_2); no longer J3.3 (Pin_3)
- net LPUART2_TX: now also J3.3 (Pin_3); no longer J3.2 (Pin_2)
- net SWCLK: now also J2.3 (Pin_3); no longer J2.4 (Pin_4)
- net SWDIO: now also J2.4 (Pin_4); no longer J2.3 (Pin_3)
Changed lines of the file:
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@@
 	)
 	(junction
+		(at 27.94 54.61)
+		(diameter 0)
+		(color 0 0 0 0)
+	)
+	(junction
 		(at 130.81 36.83)
 		(diameter 0)
@@
 	)
 	(junction
-		(at 27.94 54.61)
+		(at 27.94 71.12)
 		(diameter 0)
 		(color 0 0 0 0)
@@
 	)
 	(junction
-		(at 27.94 71.12)
-		(diameter 0)
-		(color 0 0 0 0)
-	)
-	(junction
 		(at 52.07 97.79)
 		(diameter 0)
@@
 	(wire
 		(pts
-			(xy 19.05 54.61) (xy 27.94 54.61)
-		)
-		(stroke
-			(width 0)
-			(type default)
-		)
-	)
-	(wire
-		(pts
 			(xy 109.22 55.88) (xy 111.76 55.88)
 		)
@@
 	(wire
 		(pts
-			(xy 19.05 71.12) (xy 27.94 71.12)
+			(xy 24.13 176.53) (xy 29.21 176.53)
 		)
 		(stroke
@@
 	(wire
 		(pts
-			(xy 24.13 179.07) (xy 29.21 179.07)
-		)
-		(stroke
-			(width 0)
-			(type default)
-		)
-	)
-	(wire
-		(pts
 			(xy 132.08 106.68) (xy 137.16 106.68)
 		)
@@
 	(wire
 		(pts
+			(xy 19.05 54.61) (xy 27.94 54.61)
+		)
+		(stroke
+			(width 0)
+			(type default)
+		)
+	)
+	(wire
+		(pts
 			(xy 214.63 120.65) (xy 217.17 120.65)
 		)
@@
 	(wire
 		(pts
-			(xy 24.13 176.53) (xy 29.21 176.53)
+			(xy 19.05 128.27) (xy 36.83 128.27)
 		)
 		(stroke
@@
 	(wire
 		(pts
-			(xy 19.05 128.27) (xy 36.83 128.27)
+			(xy 196.85 123.19) (xy 199.39 123.19)
 		)
 		(stroke
@@
 	(wire
 		(pts
-			(xy 196.85 123.19) (xy 199.39 123.19)
+			(xy 24.13 30.48) (xy 38.1 30.48)
 		)
 		(stroke
@@
 	(wire
 		(pts
-			(xy 24.13 30.48) (xy 38.1 30.48)
+			(xy 45.72 54.61) (xy 53.34 54.61)
 		)
 		(stroke
@@
 	(wire
 		(pts
-			(xy 45.72 54.61) (xy 53.34 54.61)
+			(xy 252.73 120.65) (xy 264.16 120.65)
 		)
 		(stroke
@@
 	(wire
 		(pts
-			(xy 252.73 120.65) (xy 264.16 120.65)
+			(xy 116.84 82.55) (xy 116.84 86.36)
 		)
 		(stroke
@@
 	(wire
 		(pts
-			(xy 116.84 82.55) (xy 116.84 86.36)
+			(xy 101.6 119.38) (xy 106.68 119.38)
 		)
 		(stroke
@@
 	(wire
 		(pts
-			(xy 101.6 119.38) (xy 106.68 119.38)
+			(xy 24.13 179.07) (xy 29.21 179.07)
 		)
 		(stroke
@@
 	(wire
 		(pts
+			(xy 19.05 71.12) (xy 27.94 71.12)
+		)
+		(stroke
+			(width 0)
+			(type default)
+		)
+	)
+	(wire
+		(pts
 			(xy 254 143.51) (xy 274.32 143.51)
 		)
@@
 		)
 	)
-	(label "LPUART2_TX"
+	(label "LPUART2_RX"
 		(at 54.61 176.53 0)
 		(effects
@@
 	)
 	(label "SWDIO"
-		(at 29.21 179.07 0)
+		(at 29.21 176.53 0)
 		(effects
 			(font
@@
 		)
 	)
-	(label "LPUART2_RX"
+	(label "LPUART2_TX"
 		(at 54.61 179.07 0)
 		(effects
@@
 	)
 	(label "SWCLK"
-		(at 29.21 176.53 0)
+		(at 29.21 179.07 0)
 		(effects
 			(font
@@
 	)
 	(symbol
+		(lib_name "R_Small_1")
 		(lib_id "Device:R_Small")
 		(at 266.7 148.59 90)
@@
 	)
 	(symbol
+		(lib_name "R_Small_3")
 		(lib_id "Device:R_Small")
 		(at 261.62 151.13 90)
@@
 	)
 	(symbol
+		(lib_name "R_Small_4")
 		(lib_id "Device:R_Small")
 		(at 250.19 120.65 90)
@@
 			)
 		)
-		(property "Footprint" "AT45DB021E-SHN-T:SOIC127P798X216-8N"
+		(property "Footprint" "XC9288A33CER-G:USP-6C"
 			(at 137.16 127.94 0)
 			(effects
@@
 	)
 	(symbol
+		(lib_name "R_Small_5")
 		(lib_id "Device:R_Small")
 		(at 255.27 123.19 90)
@@
 	)
 	(symbol
+		(lib_name "R_Small_2")
 		(lib_id "Device:R_Small")
 		(at 271.78 146.05 90)
