File: hw_rfid/hw_rfid.kicad_pcb (KiCad board)
At the start: 2 copper layers, 46 parts, among them IC1 XC9288A33CER-G, IC2 TPS610333DRLR, J1 Conn_01x02, J2 Conn_01x05, J3 Conn_01x04, J4 Conn_01x03, J5 Conn_01x08, Q1 2N7002, SW1 SW_Push, SW2 SW_Push, SW3 SW_Push, U1 STM32U031K6Ux, U2 AT45DB021E-SHN-T

Commit message: PLACA atualizada
Parts:
- IC1: footprint XC9288A:USP-6C -> XC9288A33CER-G:USP-6C
- IC2: footprint TPS6103:SOTFL50P160X60-8N -> TPS610333DRLR:SOTFL50P160X60-8N
- U2: footprint AT45DB:SOIC127P798X216-8N -> AT45DB021E-SHN-T:SOIC127P798X216-8N
- moved R7 50.2 mm to (107.1, 114.0)
- moved J1 47.8 mm to (81.8, 115.3), turned to 180 degrees
- moved C6 46.3 mm to (100.0, 99.7), turned to -90 degrees
- moved IC2 45.2 mm to (107.2, 116.8)
- moved R14 44.8 mm to (108.2, 101.5)
- moved R1 44.1 mm to (84.0, 92.9), turned to 90 degrees
- moved R5 43.6 mm to (101.0, 118.0), turned to 90 degrees
- moved R17 43.5 mm to (104.7, 101.5)
- moved R15 40.7 mm to (111.7, 101.5)
- moved L1 40.0 mm to (93.9, 121.0)
- moved J5 37.7 mm to (110.2, 105.0), turned to 90 degrees
- moved J4 37.3 mm to (141.7, 81.7)
- moved C2 35.6 mm to (104.1, 95.3), turned to -90 degrees
- moved C1 34.8 mm to (117.0, 99.5), turned to -90 degrees
- moved C7 33.0 mm to (91.5, 112.5)
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Connections:
- J2 pad 3: /SWDIO -> /SWCLK
- J2 pad 4: /SWCLK -> /SWDIO
- J3 pad 2: /LPUART2_TX -> /LPUART2_RX
- J3 pad 3: /LPUART2_RX -> /LPUART2_TX
Routing:
- net +3.3V: track 0.00 -> 265.3 mm
- net +5V: track 0.00 -> 80.5 mm, vias 0 -> 3
- net +BATT: track 0.00 -> 66.4 mm, vias 0 -> 2
- net /NRST: track 0.00 -> 38.6 mm, vias 0 -> 3
- net /ENABLE_5V_REG: track 0.00 -> 30.7 mm, vias 0 -> 3
- net /nRESET_FLASH: track 0.00 -> 30.1 mm, vias 0 -> 3
- net /AMP_PWM: track 0.00 -> 28.9 mm, vias 0 -> 3
- net /nWP_FLASH: track 0.00 -> 27.1 mm, vias 0 -> 2
- net /nRSTPD_RFID: track 0.00 -> 21.9 mm, vias 0 -> 1
- net /SWDIO: track 0.00 -> 21.8 mm
- net /SWCLK: track 0.00 -> 19.7 mm
- net /PUSH_BUTTON_01: track 0.00 -> 19.3 mm, vias 0 -> 2
- net /nCS_FLASH: track 0.00 -> 18.9 mm
- net /BOOT0: track 0.00 -> 17.6 mm
- net /SPI2_SCK_FLASH: track 0.00 -> 16.7 mm, vias 0 -> 2
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Other:
- board outline added: 70 x 60 mm

Commit message: Placa finalizada para análise
Parts:
- moved C9 11.3 mm to (97.2, 115.0)
- moved R5 4.01 mm to (97.5, 120.0)
- moved IC2 2.98 mm to (104.2, 117.2)
- moved C8 2.82 mm to (97.2, 112.4)
- moved IC1 2.70 mm to (91.5, 116.2)
- moved R7 2.42 mm to (104.7, 114.3)
- moved L1 2.39 mm to (91.9, 119.8)
- moved L2 2.37 mm to (104.6, 111.3)
- moved J3 2.06 mm to (107.7, 79.5)
- moved C10 0.96 mm to (110.6, 116.3)
- moved C7 0.36 mm to (91.9, 112.4)
- moved D1 0.10 mm to (88.9, 109.0)
Routing:
- net GND: track 0.00 -> 17.0 mm, vias 0 -> 51
- net Net-(IC1-Lx): track 12.9 -> 7.82 mm
- net +5V: track 80.5 -> 84.0 mm
- net Net-(IC2-SW): track 7.93 -> 10.5 mm
- net /ENABLE_5V_REG: track 30.7 -> 33.3 mm
- net +3.3V: track 265.3 -> 267.6 mm, vias 0 -> 2
- net +BATT: track 66.4 -> 64.1 mm
- net /LPUART2_TX: track 13.2 -> 15.3 mm
- net /LPUART2_RX: track 11.6 -> 13.7 mm
- net Net-(IC2-PG): track 7.48 -> 6.81 mm
- added copper zone on B.Cu, net GND
- added copper zone on F.Cu, net GND
Other:
- board size 70 x 60 mm -> 71.8 x 48.7 mm
