File: hw_rfid/hw_rfid.kicad_pcb (KiCad board)
At the start: 2 copper layers, 71.8 x 53.9 mm, 50 parts, among them IC1 XC9288A33CER-G, IC2 TPS610333DRLR, J1 Conn_01x02, J2 Conn_01x05, J3 Conn_01x04, J4 Conn_01x03, J5 Conn_01x08, Q1 2N7002, SW1 SW_Push, SW2 SW_Push, SW3 SW_Push, U1 STM32U031K6Ux, U2 AT45DB021E-SHN-T

Commit message: vista pelo marcelo mas nao reorganizada
Parts:
- moved J1 5.09 mm to (79.0, 111.1), turned to 0 degrees
- moved R17 3.56 mm to (108.2, 102.2)
- moved R14 3.28 mm to (111.4, 102.2)
- moved R15 2.92 mm to (114.5, 102.2)
- moved J2 2.05 mm to (119.9, 79.5)
- moved REF** 1.67 mm to (78.5, 122.7)
- moved REF** 1.56 mm to (141.2, 122.7)
- moved REF** 1.30 mm to (78.5, 76.2)
- moved REF** 1.15 mm to (141.2, 76.2)
- moved C1 0.84 mm to (116.7, 98.7)
- moved C4 0.80 mm to (115.2, 98.7)
- moved R5 0.71 mm to (97.2, 119.5)
- moved J4 0.46 mm to (141.7, 81.3)
- moved C5 0.44 mm to (105.5, 95.2)
- moved R2 0.17 mm to (100.4, 92.9)
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Routing:
- net +3.3V: track 267.6 -> 256.1 mm, vias 2 -> 6
- net GND: track 22.4 -> 16.6 mm, vias 53 -> 77
- net /nRESET_FLASH: track 30.1 -> 24.9 mm
- net Net-(J5-Pin_2): track 9.60 -> 4.93 mm
- net /SPI1_MISO_RFID: track 8.73 -> 4.32 mm, vias 2 -> 0
- net +BATT: track 64.1 -> 60.1 mm
- net /SPI1_MOSI_RFID: track 3.68 -> 6.42 mm
- net /SPI1_SCK_RFID: track 8.86 -> 6.21 mm
- net /SWDIO: track 21.8 -> 23.9 mm
- net /SWCLK: track 19.7 -> 21.8 mm
- net /NRST: track 38.6 -> 40.6 mm
- net Net-(IC2-PG): track 6.81 -> 8.71 mm
- net Net-(J5-Pin_3): track 4.66 -> 2.76 mm
- net Net-(D1-A): track 11.1 -> 9.61 mm
- net Net-(J5-Pin_4): track 10.7 -> 9.97 mm
Other:
- board size 71.8 x 53.9 mm -> 69.3 x 52.7 mm

Commit message: Finalmente finalizada para sempre
Parts:
- moved C10 2.18 mm to (109.7, 114.3)
- moved D3 0.58 mm to (102.5, 88.6)
- moved R4 0.58 mm to (107.0, 88.6)
- moved J1 0.50 mm to (79.0, 111.6)
- moved R13 0.40 mm to (121.9, 95.2)
- moved C7 0.30 mm to (91.9, 112.1)
- moved J3 0.23 mm to (107.4, 79.5)
- moved R11 0.23 mm to (121.9, 93.0)
- moved R17 0.08 mm to (108.2, 102.2)
Routing:
- net +3.3V: track 256.1 -> 250.9 mm, vias 6 -> 8
- net GND: track 16.6 -> 14.5 mm, vias 77 -> 81
- net +BATT: track 60.1 -> 58.9 mm
- net /SPI1_MOSI_RFID: track 6.42 -> 5.46 mm
- net /SPI1_SCK_RFID: track 6.21 -> 5.30 mm
- net /LED_01: track 9.97 -> 9.23 mm
- net Net-(U2-SO): track 16.6 -> 17.3 mm
- net /NRST: track 40.6 -> 39.9 mm
- net Net-(D1-A): track 9.61 -> 9.02 mm
- added copper zone on F.Cu, net +3.3V

Commit message: Final pt2 o inimigo agora é outro
Routing:
- net +5V: vias 4 -> 5
- added copper zone on F.Cu, net +5V
Changed lines of the file:
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@@
 		)
 		(embedded_fonts no)
-		(model "${KICAD9_3DMODEL_DIR}/AT45DB021E-SHN-T.3dshapes/AT45DB021E-SHN-T.step"
+		(model "${KIPRJMOD}/LIBS/AT45DB021E-SHN-T/AT45DB021E-SHN-T.step"
 			(offset
 				(xyz 0 0 0)
@@
 			)
 		)
+		(model "${KIPRJMOD}/LIBS/XC9288A33CER-G/3D/XC9288A33CER-G.stp"
+			(offset
+				(xyz 0 0 0)
+			)
+			(scale
+				(xyz 1 1 1)
+			)
+			(rotate
+				(xyz -0 -0 -0)
+			)
+		)
 	)
 	(footprint "Diode_SMD:D_SMA"
@@
 			)
 		)
+		(model "${KIPRJMOD}/LIBS/TPS610333DRLR/3D/TPS610333DRLR.stp"
+			(offset
+				(xyz 0 0 0)
+			)
+			(scale
+				(xyz 1 1 1)
+			)
+			(rotate
+				(xyz 0 0 0)
+			)
+		)
 	)
 	(footprint "Resistor_SMD:R_0603_1608Metric"
@@
 	)
 	(via
+		(at 105.169322 115.672974)
+		(size 0.508)
+		(drill 0.254)
+		(layers "F.Cu" "B.Cu")
+		(free yes)
+		(net 4)
+	)
+	(via
 		(at 138.35 84.2)
 		(size 0.508)
@@
 	)
 	(zone
-		(net 1)
-		(net_name "GND")
+		(net 4)
+		(net_name "+5V")
 		(layers "F.Cu" "B.Cu")
 		(hatch edge 0.5)
+		(priority 2)
 		(connect_pads yes
-			(clearance 0.381)
+			(clearance 0.508)
 		)
-		(min_thickness 0.254)
+		(min_thickness 0.25)
 		(filled_areas_thickness no)
 		(fill yes
-			(thermal_gap 0.508)
-			(thermal_bridge_width 0.508)
+			(thermal_gap 0.5)
+			(thermal_bridge_width 0.5)
 		)
 		(polygon
 			(pts
-				(xy 75.275 73.175) (xy 144.55 73.1) (xy 144.55 125.8) (xy 75.25 125.8)
+				(xy 103 115.589564) (xy 106.475 115.589564) (xy 106.475 118.45) (xy 103 118.45)
 			)
 		)
 	)
 	(zone
-		(net 4)
-		(net_name "+5V")
-		(layer "B.Cu")
+		(net 1)
+		(net_name "GND")
+		(layers "F.Cu" "B.Cu")
 		(hatch edge 0.5)
-		(priority 2)
-		(connect_pads
-			(clearance 0.508)
+		(connect_pads yes
+			(clearance 0.381)
 		)
-		(min_thickness 0.25)
+		(min_thickness 0.254)
 		(filled_areas_thickness no)
 		(fill yes
-			(thermal_gap 0.5)
-			(thermal_bridge_width 0.5)
+			(thermal_gap 0.508)
+			(thermal_bridge_width 0.508)
 		)
 		(polygon
 			(pts
-				(xy 103 115.675) (xy 106.475 115.675) (xy 106.475 118.45) (xy 103 118.45)
+				(xy 75.275 73.175) (xy 144.55 73.1) (xy 144.55 125.8) (xy 75.25 125.8)
 			)
 		)
