File: hw_rfid/_autosave-hw_rfid.kicad_pcb (KiCad board)
At the start: 2 copper layers, 71.8 x 53.9 mm, 50 parts, among them IC1 XC9288A33CER-G, IC2 TPS610333DRLR, J1 Conn_01x02, J2 Conn_01x05, J3 Conn_01x04, J4 Conn_01x03, J5 Conn_01x08, Q1 2N7002, SW1 SW_Push, SW2 SW_Push, SW3 SW_Push, U1 STM32U031K6Ux, U2 AT45DB021E-SHN-T

Commit message: modificações placa
Routing:
- net +BATT: track 64.1 -> 57.2 mm
- net Net-(IC2-PG): track 6.81 -> 7.80 mm
